File: ql_trump_v2_disk_interface.kicad_pcb (KiCad board)
At the start: 2 copper layers, 162.6 x 99.1 mm, 64 parts, among them J1 QL_SLOT_DIN41612_CARD, J2 Conn_02x17_Odd_Even, J3 Conn_01x01, J4 Conn_01x01, J5 Conn_01x01, U1 GAL16V8, U10 M514256A, U11 M514256A, U12 M514256A, U14 27C128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

Commit message: update BOM and gervers
Parts:
- renumbered U to U13

Commit message: update BOM and gervers
Parts:
- C1, C10, C12, C13, C15, C17, C18, C19, C20, C21, C22: value C -> 330n
- C14, C16, C23, C24, C25: value C_Polarized -> 33uF/16V
Routing:
- net /CLK: track 137.0 -> 141.2 mm
- net /CAS: track 121.2 -> 119.6 mm

Commit message: fix ROM reference
Parts:
- U14: value 27C128 -> 27C256
Changed lines of the file:
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@@
 	(title_block
 		(title "Trump Card 2 (Clone)")
-		(date "2022-10-01")
+		(date "2024-08-13")
 		(rev "01")
 		(company "Repro by Alvaro Alea Fdz.")
@@
 			)
 		)
-		(property "Value" "27C128"
+		(property "Value" "27C256"
 			(at 7.62 35.35 -90)
 			(layer "F.Fab")

Commit message: some updated on GALs
Changed lines of the file:
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@@
 		)
 		(height -3.9751)
-		(gr_text "6,4000 in"
+		(gr_text "162,5600 mm"
 			(at 120.142 39.1979 0)
 			(layer "Cmts.User")
@@
 		)
 		(height -13.335)
-		(gr_text "3,9000 in"
+		(gr_text "99,0600 mm"
 			(at 213.607 93.853 90)
 			(layer "Cmts.User")
@@
 	)
 	(segment
-		(start 116.3652 93.3781)
-		(end 126.746 82.9973)
+		(start 116.365 93.218)
+		(end 116.5253 93.218)
 		(width 0.35)
 		(layer "B.Cu")
@@
 	)
 	(segment
-		(start 126.746 75.057)
-		(end 126.497 74.808)
-		(width 0.35)
-		(layer "B.Cu")
-		(net 28)
-	)
-	(segment
 		(start 112.014 137.795)
 		(end 109.474 140.335)
@@
 	)
 	(segment
-		(start 116.365 93.218)
-		(end 116.3652 93.3781)
-		(width 0.35)
-		(layer "B.Cu")
-		(net 28)
-	)
-	(segment
 		(start 71.12 83.693)
 		(end 71.12 75.311)
@@
 	)
 	(segment
+		(start 126.497 74.808)
+		(end 126.497 74.798)
+		(width 0.35)
+		(layer "B.Cu")
+		(net 28)
+	)
+	(segment
 		(start 62.992 140.335)
 		(end 62.357 139.573)
@@
 	)
 	(segment
+		(start 116.5253 93.218)
+		(end 126.746 82.9973)
+		(width 0.35)
+		(layer "B.Cu")
+		(net 28)
+	)
+	(segment
 		(start 62.357 139.573)
 		(end 62.357 124.333)
@@
 	)
 	(segment
-		(start 126.746 82.9973)
-		(end 126.746 75.057)
+		(start 71.12 75.311)
+		(end 70.612 74.803)
 		(width 0.35)
 		(layer "B.Cu")
@@
 	)
 	(segment
-		(start 71.12 75.311)
-		(end 70.612 74.803)
+		(start 126.746 75.057)
+		(end 126.497 74.808)
 		(width 0.35)
 		(layer "B.Cu")
@@
 	)
 	(segment
-		(start 126.497 74.808)
-		(end 126.497 74.798)
+		(start 61.087 120.523)
+		(end 61.087 123.063)
 		(width 0.35)
 		(layer "B.Cu")
@@
 	)
 	(segment
-		(start 61.087 120.523)
-		(end 61.087 123.063)
+		(start 126.497 74.798)
+		(end 125.222 74.798)
 		(width 0.35)
 		(layer "B.Cu")
@@
 	)
 	(segment
-		(start 126.497 74.798)
-		(end 125.222 74.798)
+		(start 80.772 93.218)
+		(end 71.12 83.693)
 		(width 0.35)
 		(layer "B.Cu")
@@
 	)
 	(segment
-		(start 80.772 93.218)
-		(end 71.12 83.693)
+		(start 126.746 82.9973)
+		(end 126.746 75.057)
 		(width 0.35)
 		(layer "B.Cu")
@@
 		(polygon
 			(pts
-				(xy 145.034 82.931) (xy 145.049354 92.048527) (xy 139.715342 92.125106) (xy 139.7 106.553) (xy 145.034 106.553)
-				(xy 145.034 114.935) (xy 106.68 114.935) (xy 106.68 111.633) (xy 124.46 111.37926) (xy 124.4601 108.83926)
-				(xy 117.856 108.839) (xy 117.856778 91.569967) (xy 79.499718 91.686024) (xy 79.496858 90.679526)
-				(xy 66.548 90.720468) (xy 66.548 86.233) (xy 64.262 83.947) (xy 61.982629 83.947707) (xy 61.978924 76.073716)
-				(xy 53.593328 76.073336) (xy 53.593739 72.263) (xy 42.419319 72.263059) (xy 42.419524 66.928127)
-				(xy 56.640996 66.929) (xy 56.639575 53.984053) (xy 67.815575 53.981731) (xy 67.818 79.121) (xy 141.732 79.121)
+				(xy 145.034 82.931) (xy 145.049354 92.048527) (xy 139.715342 92.125106) (xy 139.7 94.615) (xy 123.444 94.615)
+				(xy 123.444 105.918) (xy 145.034 105.918) (xy 145.034 114.935) (xy 106.68 114.935) (xy 106.68 111.633)
+				(xy 124.46 111.37926) (xy 124.4601 108.83926) (xy 117.856 108.839) (xy 117.856778 91.569967) (xy 79.499718 91.686024)
+				(xy 79.496858 90.679526) (xy 66.548 90.720468) (xy 66.548 86.233) (xy 64.262 83.947) (xy 61.982629 83.947707)
+				(xy 61.978924 76.073716) (xy 53.593328 76.073336) (xy 53.593739 72.263) (xy 42.419319 72.263059)
+				(xy 42.419524 66.928127) (xy 56.640996 66.929) (xy 56.639575 53.984053) (xy 67.815575 53.981731)
+				(xy 67.818 79.121) (xy 141.732 79.121)
 			)
 		)
@@
 			)
 		)
+	)
+	(zone
+		(net 0)
+		(net_name "")
+		(layer "F.Cu")
+		(hatch edge 0.5)
+		(connect_pads
+			(clearance 0)
+		)
+		(min_thickness 0.25)
+		(filled_areas_thickness no)
+		(keepout
+			(tracks not_allowed)
+			(vias not_allowed)
+			(pads not_allowed)
+			(copperpour not_allowed)
+			(footprints allowed)
+		)
+		(fill
+			(thermal_gap 0.5)
+			(thermal_bridge_width 0.5)
+		)
+		(polygon
+			(pts
+				(xy 131.064 108.458) (xy 131.064 112.903) (xy 134.493 112.903) (xy 134.493 108.458)
+			)
+		)

Commit message: minor typos
Parts:
- J1: footprint Connector_DIN:DIN41612_B_2x32_Male_Horizontal_THT -> Connector_DIN:DIN41612_Q_2x32_Female_Horizontal_THT
Connections:
- net Net-(D4-K) renamed /GAL2_P11

Commit message: new devel branch
Parts:
- U1, U2: value GAL16V8 -> GAL16V8-15
- U15: value 74HC04 -> 7416N
- U16: value 74LS175 -> 74F175N
- U17: value 74ls175 -> 74F175N
- U3: value 74HC04 -> 74HC04N
- U5, U6: value 74LS157 -> 74HC257N
- moved R5 10.2 mm to (152.7, 123.6), turned to 180 degrees
- moved R6 10.2 mm to (152.7, 126.1), turned to 180 degrees
- moved C4 4.42 mm to (173.8, 123.6), turned to 180 degrees
- moved J5 1.11 mm to (162.6, 54.3)
- moved J4 0.82 mm to (172.1, 54.3)
- moved J3 0.81 mm to (168.4, 54.3)
- moved U4 0.69 mm to (185.9, 66.5)
- moved R3 0.13 mm to (162.8, 136.4)
Connections:
- net /GAL2_P11 renamed /T3
- net /GAL2_P15 renamed /T1
- net /GAL2_P9 renamed /T2
- net Net-(D2-K) renamed /DTACK2L
- net Net-(D3-K) renamed /DTACK1L
- net Net-(U1-IO7) renamed /P13
- U10 pad 1: /D4 -> /D6
- U10 pad 18: /D6 -> /D4
- U10 pad 19: /D7 -> /D5
- U10 pad 2: /D5 -> /D7
- U10 pad 4: /RAS1 -> /RAS2
- U11 pad 1: /D0 -> /D7
- U11 pad 18: /D2 -> /D5
- U11 pad 19: /D3 -> /D4
- U11 pad 2: /D1 -> /D6
- U12 pad 1: /D4 -> /D3
- U12 pad 18: /D6 -> /D1
- U12 pad 19: /D7 -> /D0
- U12 pad 2: /D5 -> /D2
- U16 pad 11: unconnected-(U16-~{Q2}-Pad11) -> /DS2
- U16 pad 12: /D7 -> /D5
- U16 pad 13: /D6 -> /D4
- U16 pad 14: unconnected-(U16-~{Q3}-Pad14) -> /DS3
- U16 pad 3: /DS3 -> unconnected-(U16-~{Q0}-Pad3)
- U16 pad 4: /D4 -> /D6
- U16 pad 5: /D5 -> /D7
- U16 pad 6: /DS2 -> unconnected-(U16-~{Q1}-Pad6)
- U17 pad 11: /MOTOR_ON -> /HEAD
- U17 pad 12: /D2 -> /D3
- U17 pad 3: /HEAD -> /MOTOR_ON
- U17 pad 4: /D3 -> /D2
- U7 pad 4: /RAS2 -> /RAS1
- U8 pad 4: /RAS2 -> /RAS1
- U9 pad 1: /D0 -> /D1
- U9 pad 2: /D1 -> /D0
- U9 pad 4: /RAS1 -> /RAS2
Routing:
- net /A9: track 220.9 -> 124.1 mm, vias 5 -> 2
- net /RAS1: track 128.7 -> 79.5 mm, vias 5 -> 0
- net /D0: track 302.3 -> 348.5 mm, vias 3 -> 5
- net /A4: track 141.7 -> 97.9 mm, vias 4 -> 0
- net /DATA_WR: track 71.3 -> 112.4 mm, vias 1 -> 2
- net /RAS2: track 69.4 -> 110.5 mm, vias 2 -> 1
- net /GATE_WR: track 80.3 -> 121.2 mm, vias 1 -> 0
- net /DS3: track 64.8 -> 24.6 mm, vias 1 -> 0
- net /DSMC: track 77.5 -> 38.5 mm, vias 0 -> 1
- net /A1: track 176.8 -> 138.5 mm, vias 5 -> 1
- net /DS2: track 63.0 -> 27.4 mm, vias 1 -> 2
- net /A12: track 75.8 -> 108.7 mm, vias 3 -> 1
- net /A2: track 136.8 -> 105.9 mm, vias 6 -> 1
- net GND: track 961.8 -> 992.5 mm, vias 5 -> 8
- net /A3: track 131.8 -> 101.4 mm, vias 3 -> 0
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Other:
- board text added: "34"
- board text added: "CARD"
- board text added: "DS4"
- board text added: "DS5"
- board text added: "TRUMP"
- board text removed: "TRUMP CARD"

Commit message: small details
Parts:
- C13, C15: footprint Capacitor_THT:C_Disc_D5.1mm_W3.2mm_P5.00mm -> Capacitor_THT:C_Disc_D5.0mm_W2.5mm_P5.00mm
- moved J2 0.51 mm to (51.6, 114.4)
- moved C15 0.38 mm to (41.3, 59.8)
- moved C13 0.22 mm to (55.0, 59.8)
- moved U18 0.13 mm to (45.6, 64.8)
- moved C23 0.12 mm to (92.2, 54.5)
- moved C24 0.12 mm to (120.1, 54.6)
Routing:
- net +5V: track 816.6 -> 818.3 mm
- net /MOTOR_ON: track 51.9 -> 53.4 mm
- net /STEP: track 88.8 -> 89.9 mm
- net /GATE_WR: track 121.2 -> 122.0 mm
- net /DS1: track 29.3 -> 30.1 mm
- net /DIR: track 95.2 -> 95.9 mm
- net /CAS: track 147.6 -> 148.2 mm
- net /D0: track 348.5 -> 347.9 mm
- net /FDC_RD: track 80.6 -> 81.1 mm
- net /DS3: track 24.6 -> 25.1 mm
- net /DS2: track 27.4 -> 27.9 mm
- net /ROM_OE: track 59.8 -> 59.3 mm
Other:
- outline, holes or cut-outs redrawn
- board text added: "♠"
- board text added: "♣"
- board text added: "♥"
- board text added: "♦"
