File: ql_trump_v2_disk_interface.kicad_sch (KiCad schematic)
At the start: 64 parts, among them J1 QL_SLOT_DIN41612_CARD, J2 Conn_02x17_Odd_Even, J3 Conn_01x01, J4 Conn_01x01, J5 Conn_01x01, U1 GAL16V8, U10 M514256A, U11 M514256A, U12 M514256A, U14 27C128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

Commit message: update BOM and gervers
Parts:
- C1, C10, C12, C13, C15, C17, C18, C19, C20, C21, C22: value C -> 330n
- C14, C16, C23, C24, C25: value C_Polarized -> 33uF/16V
- renumbered U to U13
Other:
- note added: "NOTE: C1,C10,C12,C15,C17 to C22 to C10 is in some photos 100nF (104 disc or yellow) and in another 330nF (330n blue) value is not critical. C14,C16,C23-C25 are also no critical, and size shall be checked as can conflict with memory chips and 7805, consider use 33uF/25V for C14"

Commit message: fix ROM reference
Parts:
- U14: value 27C128 -> 27C256
Other:
- note added: "NOTE: C1,C10,C12,C15,C17 to C22 to C10 is in some photos 100nF (104 disc or yellow) and in another 330nF (330n blue) value is not critical. C14,C16,C23-C25 are also no critical, and size shall be checked as can conflict with memory chips and 7805, consider use 33uF/25V for C14 U14 is originally a 32Kb EPROM (UV Erasable) but a W27C512 (64Kb EEPROM) will work, if you burn the ROM image in the top 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"
- note removed: "NOTE: C1,C10,C12,C15,C17 to C22 to C10 is in some photos 100nF (104 disc or yellow) and in another 330nF (330n blue) value is not critical. C14,C16,C23-C25 are also no critical, and size shall be checked as can conflict with memory chips and 7805, consider use 33uF/25V for C14"
Changed lines of the file:
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@@
 	(title_block
 		(title "Trump Card 2 (Clone)")
-		(date "2024-07-26")
+		(date "2024-08-13")
 		(rev "01")
 		(company "Repro by Alvaro Alea Fdz.")
@@
 		)
 	)
-	(text "NOTE:\n\nC1,C10,C12,C15,C17 to C22 to C10 is in some photos 100nF (104 disc or yellow) \nand in another 330nF (330n blue) value is not critical.\n\nC14,C16,C23-C25 are also no critical, and size shall be checked as can conflict \nwith memory chips and 7805, consider use 33uF/25V for C14\n\n"
+	(text "NOTE:\n\nC1,C10,C12,C15,C17 to C22 to C10 is in some photos 100nF (104 disc or yellow) \nand in another 330nF (330n blue) value is not critical.\n\nC14,C16,C23-C25 are also no critical, and size shall be checked as can conflict\nwith memory chips and 7805, consider use 33uF/25V for C14\n\nU14 is originally a 32Kb EPROM (UV Erasable) but a W27C512 (64Kb EEPROM) will work, if\nyou burn the ROM image in the top 32Kb of the memory. \n\n\n"
 		(exclude_from_sim no)
-		(at 478.536 365.506 0)
+		(at 475.996 358.394 0)
 		(effects
 			(font
@@
 		(fields_autoplaced yes)
 		(property "Reference" "U14"
-			(at 156.9594 31.115 0)
+			(at 157.1341 31.75 0)
 			(effects
 				(font
@@
 			)
 		)
-		(property "Value" "27C128"
-			(at 156.9594 33.655 0)
+		(property "Value" "27C256"
+			(at 157.1341 34.29 0)
 			(effects
 				(font

Commit message: some updated on GALs
Other:
- note added: "(T1)"
- note added: "(T2)"
- note added: "(T3)"
- note added: "BANK for 256, 512,768"
- note added: "BANK for 512,768"
- note added: "BANK for 768, ACE"
Changed lines of the file:
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@@
 	(title_block
 		(title "Trump Card 2 (Clone)")
-		(date "2024-08-13")
-		(rev "01")
+		(date "2024-11-11")
+		(rev "1.1")
 		(company "Repro by Alvaro Alea Fdz.")
 		(comment 1 "Disk Interface for Sinclair QL")
@@
 		)
 	)
+	(text "(T1)"
+		(exclude_from_sim no)
+		(at 286.512 215.646 0)
+		(effects
+			(font
+				(size 1.27 1.27)
+			)
+		)
+	)
 	(text "NOTE:\n\nC1,C10,C12,C15,C17 to C22 to C10 is in some photos 100nF (104 disc or yellow) \nand in another 330nF (330n blue) value is not critical.\n\nC14,C16,C23-C25 are also no critical, and size shall be checked as can conflict\nwith memory chips and 7805, consider use 33uF/25V for C14\n\nU14 is originally a 32Kb EPROM (UV Erasable) but a W27C512 (64Kb EEPROM) will work, if\nyou burn the ROM image in the top 32Kb of the memory. \n\n\n"
 		(exclude_from_sim no)
@@
 		)
 	)
+	(text "BANK for 512,768"
+		(exclude_from_sim no)
+		(at 460.756 187.96 0)
+		(effects
+			(font
+				(size 1.27 1.27)
+			)
+		)
+	)
+	(text "(T2)"
+		(exclude_from_sim no)
+		(at 310.134 234.188 0)
+		(effects
+			(font
+				(size 1.27 1.27)
+			)
+		)
+	)
 	(text "DS0\n"
 		(exclude_from_sim no)
@@
 		)
 	)
+	(text "(T3)"
+		(exclude_from_sim no)
+		(at 57.912 222.504 0)
+		(effects
+			(font
+				(size 1.27 1.27)
+			)
+		)
+	)
 	(text "Only Install for with RAM chips"
 		(exclude_from_sim no)
@@
 		)
 	)
+	(text "BANK for 768, ACE"
+		(exclude_from_sim no)
+		(at 407.416 187.96 0)
+		(effects
+			(font
+				(size 1.27 1.27)
+			)
+		)
+	)
 	(text "N/C"
 		(exclude_from_sim no)
@@
 		)
 	)
+	(text "BANK for 256, 512,768"
+		(exclude_from_sim no)
+		(at 508.254 188.722 0)
+		(effects
+			(font
+				(size 1.27 1.27)
+			)
+		)
+	)
+	(text "(T2)"
+		(exclude_from_sim no)
+		(at 51.308 216.916 0)
+		(effects
+			(font
+				(size 1.27 1.27)
+			)
+		)
+	)

Commit message: minor typos
Parts:
- J1: footprint Connector_DIN:DIN41612_B_2x32_Male_Horizontal_THT -> Connector_DIN:DIN41612_Q_2x32_Female_Horizontal_THT
Connections:
- net GAL2_P11: now reaches C2.2, D4.1 (K), R4.1, U2.11 (I10/~{OE})
Other:
- moved on the sheet: C2, C3, C4, C5, D1, D10, D3, D4, D5, D6, D7, D9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

Commit message: new devel branch
Parts:
- U1, U2: value GAL16V8 -> GAL16V8-15
- U15: value 74HC04 -> 7416N
- U16: value 74LS175 -> 74F175N
- U17: value 74ls175 -> 74F175N
- U3: value 74HC04 -> 74HC04N
- U5, U6: value 74LS157 -> 74HC257N
Connections:
- net D0: now also U12.19 (D3), U9.2 (D1); no longer U11.1 (D0), U9.1 (D0)
- net D1: now also U12.18 (D2), U9.1 (D0); no longer U11.2 (D1), U9.2 (D1)
- net D2: now also U12.2 (D1), U17.4 (D0); no longer U11.18 (D2), U17.12 (D2)
- net D3: now also U12.1 (D0), U17.12 (D2); no longer U11.19 (D3), U17.4 (D0)
- net D4: now also U10.18 (D2), U11.19 (D3), U16.13 (D3); no longer U10.1 (D0), U12.1 (D0), U16.4 (D0)
- net D5: now also U10.19 (D3), U11.18 (D2), U16.12 (D2); no longer U10.2 (D1), U12.2 (D1), U16.5 (D1)
- net D6: now also U10.1 (D0), U11.2 (D1), U16.4 (D0); no longer U10.18 (D2), U12.18 (D2), U16.13 (D3)
- net D7: now also U10.2 (D1), U11.1 (D0), U16.5 (D1); no longer U10.19 (D3), U12.19 (D3), U16.12 (D2)
- net DS2: now also U16.11 (~{Q2}); no longer U16.6 (~{Q1})
- net DS3: now also U16.14 (~{Q3}); no longer U16.3 (~{Q0})
- net HEAD: now also U17.11 (~{Q2}); no longer U17.3 (~{Q0})
- net MOTOR_ON: now also U17.3 (~{Q0}); no longer U17.11 (~{Q2})
- net RAS1: now also U7.4 (~{RAS}), U8.4 (~{RAS}); no longer U10.4 (~{RAS}), U9.4 (~{RAS})
- net RAS2: now also U10.4 (~{RAS}), U9.4 (~{RAS}); no longer U7.4 (~{RAS}), U8.4 (~{RAS})
- net DTACK1L: now reaches D3.1 (K), U2.14 (IO6)
- net P13: now reaches U1.13 (IO7), U2.1 (I1/CLK)
- net DTACK2L: now reaches D2.1 (K), U2.16 (IO4)
- net GAL2_P11 renamed T3
- net GAL2_P15 renamed T1
- net GAL2_P9 renamed T2
Other:
- note added: "NOTE: Values are for U2 = PAL16V8 If use a GAL16V8 for U2 R2 = 470 R1 = 1K9 R4 = 960"
- note removed: "(T1)"
- note removed: "(T2)"
- note removed: "(T3)"
- moved on the sheet: C2, C3, C4, C5, D10, D4, D5, D9, R1, R2, R3, R4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

Commit message: small details
Connections:
- net GND: no longer C17.2, C18.2, C19.1, C20.2, C21.1, C22.2, C23.2, C24.2, C25.2
- new net: C17.2, C18.2, C19.1, C20.2, C21.1, C22.2, C23.2, C24.2, C25.2
Other:
- note added: "For no RAM version, replace D5, D9 and D10 by wires, or 0ohms resistors"
- note removed: "For no RAM version, replace D5, D9 and D10 by wires, or 0ohm resistors"
- moved on the sheet: C1, C10, C12, C13, C14, C15, C16, C17, C18, C19, C2, C20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
